File: hw/8088_cpu_card.kicad_pcb (KiCad board)
At the start: 2 copper layers, 97.8 x 99.6 mm, 1 part, among them J2 PC XT ISA

Commit message: kinda working revision
Parts:
- added C1: 20p XTAL, Capacitor_SMD:C_0402_1005Metric_Pad0.74x0.62mm_HandSolder, B.Cu at (102.6, 69.6)
- added C10: 100n/0.1u PWR, Capacitor_SMD:C_1206_3216Metric_Pad1.33x1.80mm_HandSolder, B.Cu at (109.6, 96.6)
- added C2: 20p XTAL, Capacitor_SMD:C_0402_1005Metric_Pad0.74x0.62mm_HandSolder, B.Cu at (103.8, 54.5)
- added C3: 1u BTN, Capacitor_SMD:C_0805_2012Metric_Pad1.18x1.45mm_HandSolder, B.Cu at (138.3, 66.4)
- added C4: PPWR, Capacitor_Tantalum_SMD:CP_EIA-7343-31_Kemet-D, B.Cu at (97.9, 124.5)
- added C5: 100n/0.1u PWR, Capacitor_SMD:C_1206_3216Metric_Pad1.33x1.80mm_HandSolder, B.Cu at (123.1, 47.4)
- added C6: 100n/0.1u PWR, Capacitor_SMD:C_1206_3216Metric_Pad1.33x1.80mm_HandSolder, B.Cu at (157.0, 48.3)
- added C7: 100n/0.1u PWR, Capacitor_SMD:C_1206_3216Metric_Pad1.33x1.80mm_HandSolder, B.Cu at (123.1, 82.0)
- added C8: 100n/0.1u PWR, Capacitor_SMD:C_1206_3216Metric_Pad1.33x1.80mm_HandSolder, B.Cu at (157.2, 91.6)
- added C9: 100n/0.1u PWR, Capacitor_SMD:C_1206_3216Metric_Pad1.33x1.80mm_HandSolder, B.Cu at (139.4, 125.7)
- added J1: 80188, 80C188:PGA68-N, F.Cu at (121.5, 64.9)
- added J3: GAL16V8, Package_DIP:DIP-20_W7.62mm, F.Cu at (155.5, 60.3)
- added J4: SST39SF020, Package_LCC:PLCC-32_11.4x14.0mm_P1.27mm, F.Cu at (158.5, 79.4)
- added J5: 8259, Package_LCC:PLCC-28_THT-Socket, F.Cu at (178.8, 107.7)
- added JP1: IRQ2, Jumper:SolderJumper-3_P1.3mm_Open_RoundedPad1.0x1.5mm, B.Cu at (170.9, 126.4)
- added JP2: IRQ3, Jumper:SolderJumper-3_P1.3mm_Open_RoundedPad1.0x1.5mm, B.Cu at (120.5, 126.5)
- added R1: PullUP, Resistor_SMD:R_1206_3216Metric_Pad1.30x1.75mm_HandSolder, F.Cu at (185.0, 67.4)
- added R2: Limit, Resistor_SMD:R_1206_3216Metric_Pad1.30x1.75mm_HandSolder, B.Cu at (107.8, 45.8)
- added R3: Limit, Resistor_SMD:R_1206_3216Metric_Pad1.30x1.75mm_HandSolder, B.Cu at (115.1, 45.8)
- added R4: Limit, Resistor_SMD:R_1206_3216Metric_Pad1.30x1.75mm_HandSolder, B.Cu at (145.0, 65.0)
- added SW1: RESET, Button_Switch_SMD:SW_SPST_EVQP7A, F.Cu at (187.3, 74.2)
- added U1: SN74ABT16841DL, SN74ABT16841DL:SOP64P1035X279-56N, F.Cu at (112.7, 97.2)
- added U2: 74LS245, Package_SO:SOIC-20W_7.5x12.8mm_P1.27mm, B.Cu at (163.8, 79.4)
- added U3: SRAM, Package_SO:SSOP-32_11.305x20.495mm_P1.27mm, F.Cu at (146.1, 111.6)
- added Y1: 16MHz, Crystal:Crystal_SMD_0603-4Pin_6.0x3.5mm_HandSoldering, B.Cu at (102.2, 62.0)
Connections:
- J2 pad 15: unconnected-(J2-Pad15) -> ~{PCS6}
- J2 pad 17: unconnected-(J2-Pad17) -> ~{PCS4}
- J2 pad 18: DRQ1 -> DRQ0
- J2 pad 19: unconnected-(J2-Pad19) -> ~{PCS3}
- J2 pad 21: unconnected-(J2-Pad21) -> IR7
- J2 pad 22: unconnected-(J2-Pad22) -> IR6
- J2 pad 23: unconnected-(J2-Pad23) -> IR5
- J2 pad 24: unconnected-(J2-Pad24) -> IR4
- J2 pad 25: unconnected-(J2-Pad25) -> IRQ3
- J2 pad 26: unconnected-(J2-Pad26) -> ~{PCS5}
- J2 pad 4: unconnected-(J2-Pad4) -> IRQ2
- J2 pad 6: unconnected-(J2-Pad6) -> DRQ1
- J2 pad 8: unconnected-(J2-Pad8) -> ~{CARDSLCTD}
Routing:
- net VCC: track 0.00 -> 542.2 mm, vias 0 -> 16
- net DA5: track 0.00 -> 233.1 mm, vias 0 -> 7
- net A0: track 0.00 -> 223.3 mm, vias 0 -> 7
- net DA2: track 0.00 -> 213.9 mm, vias 0 -> 6
- net ALE: track 0.00 -> 213.3 mm, vias 0 -> 3
- net RESET: track 0.00 -> 187.9 mm, vias 0 -> 3
- net DA0: track 0.00 -> 184.2 mm, vias 0 -> 8
- net INT1: track 0.00 -> 170.8 mm, vias 0 -> 2
- net ~{IOR}: track 0.00 -> 167.4 mm, vias 0 -> 4
- net DA3: track 0.00 -> 157.3 mm, vias 0 -> 3
- net A7: track 0.00 -> 148.5 mm, vias 0 -> 4
- net A3: track 0.00 -> 145.8 mm, vias 0 -> 5
- net DA6: track 0.00 -> 144.1 mm, vias 0 -> 3
- net A1: track 0.00 -> 140.7 mm, vias 0 -> 3
- net A6: track 0.00 -> 136.7 mm, vias 0 -> 4
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
Commit message: minimal viable board
* PLD provides /IOW and TRG signals for reading all IO out
* BIOS initialises the /UMCS and print debug
Connections:
- J3 pad 12: unconnected-(J3-Pad12) -> /TRG
Changed lines of the file:
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@@
   (net 115 "~{BDEN}")
   (net 116 "~{ALE}")
-  (net 117 "unconnected-(J3-Pad12)")
+  (net 117 "/TRG")
   (net 118 "/M{slash}~{IO}")
   (net 119 "unconnected-(J4-Pad1)")
@@
       (net 1 "GND") (pinfunction "I10/~{OE}") (pintype "input"))
     (pad "12" thru_hole oval (at 7.62 20.32 90) (size 1.6 1.6) (drill 0.8) (layers *.Cu *.Mask)
-      (net 117 "unconnected-(J3-Pad12)") (pinfunction "IO8") (pintype "tri_state+no_connect"))
+      (net 117 "/TRG") (pinfunction "IO8") (pintype "tri_state"))
     (pad "13" thru_hole oval (at 7.62 17.78 90) (size 1.6 1.6) (drill 0.8) (layers *.Cu *.Mask)
       (net 10 "~{IOR}") (pinfunction "IO7") (pintype "tri_state"))
